Commit message: Commit 1-2: Foundation Setup - Enhanced robot description with Gazebo integration
- Added clean robot URDF with collision and inertial properties
- Created conveyor belt system with physics simulation
- Implemented robot controller with smooth joint interpolation
- Added Gazebo integration with ROS 2 control
- Created comprehensive launch files for testing
- Added professional documentation without emojis
- Established modular package architecture
- Timeline: January 2025 - Phase 1 Foundation Setup

Developer: Sai-04021210 (inthedarkshades00008@gmail.com)
Project: Conveyor Belt Pick-and-Place Robot System

File: install/basic_description/share/basic_description/urdf/basic_urdf.xacro (robot description, xacro)
@@ -11,5 +11,19 @@
                 <mesh filename="package://basic_description/meshes/basement.STL" scale="0.01 0.01 0.01"/>
             </geometry>
+            <material name="base_material">
+                <color rgba="0.5 0.5 0.5 1.0"/>
+            </material>
         </visual>
+        <collision>
+            <origin rpy="0 0 0" xyz="-0.5 -0.5 0"/>
+            <geometry>
+                <mesh filename="package://basic_description/meshes/basement.STL" scale="0.01 0.01 0.01"/>
+            </geometry>
+        </collision>
+        <inertial>
+            <origin xyz="0 0 0.15" rpy="0 0 0"/>
+            <mass value="5.0"/>
+            <inertia ixx="0.1" ixy="0" ixz="0" iyy="0.1" iyz="0" izz="0.1"/>
+        </inertial>
     </link>
     <joint name="virtual_joint" type="fixed">
@@ -24,5 +38,19 @@
                 <mesh filename="package://basic_description/meshes/base_plate.STL" scale="0.01 0.01 0.01"/>
             </geometry>
+            <material name="baseplate_material">
+                <color rgba="0.2 0.2 0.8 1.0"/>
+            </material>
         </visual>
+        <collision>
+            <origin rpy="0 0 0" xyz="-0.39 -0.39 -0.56"/>
+            <geometry>
+                <mesh filename="package://basic_description/meshes/base_plate.STL" scale="0.01 0.01 0.01"/>
+            </geometry>
+        </collision>
+        <inertial>
+            <origin xyz="0 0 0" rpy="0 0 0"/>
+            <mass value="2.0"/>
+            <inertia ixx="0.05" ixy="0" ixz="0" iyy="0.05" iyz="0" izz="0.05"/>
+        </inertial>
     </link>
     <joint name="baseplate_joint" type="revolute">
